Commit message: Created copy of urdf to test with and created simple simulation visualization in Julia

File: kortex_description/arms/gen3/7dof/urdf/GEN3_URDF_V12 copy.urdf (robot description, URDF)
Before this commit: robot GEN3_URDF_V12, 9 links, 8 joints
Links:
- link Bracelet_Link: geometry collision mesh filename=/home/amkyu/catkin_workspace/src/ros_kortex/kortex_descript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; visual mesh filename=/home/amkyu/catkin_workspace/src/ros_kortex/kortex_descript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
- link ForeArm_Link: geometry collision mesh filename=/home/amkyu/catkin_workspace/src/ros_kortex/kortex_descript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; visual mesh filename=/home/amkyu/catkin_workspace/src/ros_kortex/kortex_descript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
- link HalfArm1_Link: geometry collision mesh filename=/home/amkyu/catkin_workspace/src/ros_kortex/kortex_descript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; visual mesh filename=/home/amkyu/catkin_workspace/src/ros_kortex/kortex_descript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
- link HalfArm2_Link: geometry collision mesh filename=/home/amkyu/catkin_workspace/src/ros_kortex/kortex_descript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; visual mesh filename=/home/amkyu/catkin_workspace/src/ros_kortex/kortex_descript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
- link Shoulder_Link: geometry collision mesh filename=/home/amkyu/catkin_workspace/src/ros_kortex/kortex_descript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; visual mesh filename=/home/amkyu/catkin_workspace/src/ros_kortex/kortex_descript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
- link SphericalWrist1_Link: geometry collision mesh filename=/home/amkyu/catkin_workspace/src/ros_kortex/kortex_descript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; visual mesh filename=/home/amkyu/catkin_workspace/src/ros_kortex/kortex_descript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
- link SphericalWrist2_Link: geometry collision mesh filename=/home/amkyu/catkin_workspace/src/ros_kortex/kortex_descript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; visual mesh filename=/home/amkyu/catkin_workspace/src/ros_kortex/kortex_descript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
- link base_link: geometry collision mesh filename=/home/amkyu/catkin_workspace/src/ros_kortex/kortex_descript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; visual mesh filename=/home/amkyu/catkin_workspace/src/ros_kortex/kortex_descript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
