Commit message: update urdf and moveit config

File: kortex_description/arms/gen3/7dof/urdf/gen3_macro.xacro (robot description, xacro)
@@ -298,5 +298,36 @@
         velocity="1.2218" />
     </joint>
-    <link name="${prefix}ftsensor_link">
+    <link name="${prefix}ee_adapter_link">
+      <inertial>
+        <origin xyz="-9.3E-05 0.000132 -0.022905" rpy="0 0 0" />
+        <mass value="0.130" />
+        <inertia ixx="0.000214" ixy="0" ixz="1E-06" iyy="0.000223" iyz="-2E-06" izz="0.00024" />
+      </inertial>
+      <visual>
+        <origin xyz="-0.04 -0.04 0" rpy="0 0 0" />
+        <geometry>
+          <mesh filename="package://kortex_description/arms/gen3/${dof}dof/meshes/ReamerAssemblyCombine.stl" scale="0.001 0.001 0.001"/>
+        </geometry>
+        <material name="">
+          <color rgba="0.75294 0.75294 0.75294 1" />
+        </material>
+      </visual>
+      <collision>
+        <origin xyz="-0.04 -0.04 0" rpy="0 0 0" />
+        <geometry>
+          <mesh filename="package://kortex_description/arms/gen3/${dof}dof/meshes/ReamerAssemblyCombine.stl" scale="0.001 0.001 0.001"/>
+        </geometry>
+      </collision>
+    </link>
+    <joint name="${prefix}ee_joint" type="fixed">
+      <origin xyz="0 0 -0.0615250000000001" rpy="3.14159265358979 1.09937075168372E-32 0" />
+      <parent
+        link="${prefix}bracelet_link" />
+      <child
+        link="${prefix}ee_adapter_link" />
+      <axis
+        xyz="0 0 0" />
+    </joint>
+    <!-- <link name="${prefix}ftsensor_link">
       <inertial>
         <origin xyz="-9.3E-05 0.000132 -0.022905" rpy="0 0 0" />
@@ -383,9 +414,10 @@
       <axis
         xyz="0 0 0" />
-    </joint>
-    <!-- <joint
+    </joint> -->
+    <link name="${prefix}end_effector_link" />
+    <joint
       name="${prefix}end_effector"
       type="fixed">
-      <origin xyz="0 0 -0.0615250000000001" rpy="3.14159265358979 1.09937075168372E-32 0" />
+      <origin xyz="0 0 0.29990848" rpy="0 0 0" />
       <parent
         link="${prefix}ee_adapter_link" />
@@ -394,6 +426,6 @@
       <axis
         xyz="0 0 0" />
-    </joint> -->
-     <joint
+    </joint>
+     <!-- <joint
       name="${prefix}reamer_link"
       type="fixed">
@@ -417,5 +449,5 @@
       <axis
         xyz="0 0 0" />
-    </joint>
+    </joint> -->
     <!-- <xacro:if value="${vision}">
       <link name="${prefix}camera_link" />
@@ -438,5 +470,5 @@
       </joint>
     </xacro:if> -->
-    <gazebo reference="${prefix}ft_sensor">
+    <!-- <gazebo reference="${prefix}ft_sensor">
         <provideFeedback>true</provideFeedback>
         <disableFixedJointLumping>true</disableFixedJointLumping>
@@ -449,5 +481,5 @@
             <jointName>${prefix}ft_sensor</jointName>
         </plugin>
-    </gazebo>
+    </gazebo> -->
   </xacro:macro>
 </robot>

File: kortex_move_it_config/gen3_move_it_config/config/7dof/gen3.srdf.xacro (robot description, xacro)
@@ -1,9 +1,8 @@
-<?xml version="1.0" ?>
+<?xml version="1.0" encoding="UTF-8"?>
 <!--This does not replace URDF, and is not an extension of URDF.
     This is a format for representing semantic information about the robot structure.
     A URDF file must exist for this robot as well, where the joints and the links that are referenced are defined
 -->
-<robot name="gen3" xmlns:xacro="http://www.ros.org/wiki/xacro">
-    <xacro:arg name="prefix" default="" />
+<robot name="gen3">
     <!--GROUPS: Representation of a set of joints and links. This can be useful for specifying DOF to plan for, defining arms, end effectors, etc-->
     <!--LINKS: When a link is specified, the parent joint of that link (if it exists) is automatically included-->
@@ -12,68 +11,65 @@
     <!--SUBGROUPS: Groups can also be formed by referencing to already defined group names-->
     <group name="arm">
-        <joint name="$(arg prefix)joint_1" />
-        <joint name="$(arg prefix)joint_2" />
-        <joint name="$(arg prefix)joint_3" />
-        <joint name="$(arg prefix)joint_4" />
-        <joint name="$(arg prefix)joint_5" />
-        <joint name="$(arg prefix)joint_6" />
-        <joint name="$(arg prefix)joint_7" />
-        <joint name="$(arg prefix)end_effector" />
-        <joint name="$(arg prefix)tool_frame_joint" />
+        <joint name="world_frame"/>
+        <joint name="joint_1"/>
+        <joint name="joint_2"/>
+        <joint name="joint_3"/>
+        <joint name="joint_4"/>
+        <joint name="joint_5"/>
+        <joint name="joint_6"/>
+        <joint name="joint_7"/>
+    </group>
+    <group name="reamer">
+        <joint name="ee_joint"/>
+        <joint name="end_effector"/>
+        <joint name="tool_frame_joint"/>
     </group>
     <!--GROUP STATES: Purpose: Define a named state for a particular group, in terms of joint values. This is useful to define states like 'folded arms'-->
     <group_state name="home" group="arm">
-        <joint name="$(arg prefix)joint_1" value="0" />
-        <joint name="$(arg prefix)joint_2" value="0.26" />
-        <joint name="$(arg prefix)joint_3" value="3.14" />
-        <joint name="$(arg prefix)joint_4" value="-2.27" />
-        <joint name="$(arg prefix)joint_5" value="0" />
-        <joint name="$(arg prefix)joint_6" value="0.96" />
-        <joint name="$(arg prefix)joint_7" value="1.57" />
-    </group_state>
-    <group_state name="retract" group="arm">
-        <joint name="$(arg prefix)joint_1" value="0" />
-        <joint name="$(arg prefix)joint_2" value="-0.35" />
-        <joint name="$(arg prefix)joint_3" value="3.14" />
-        <joint name="$(arg prefix)joint_4" value="-2.54" />
-        <joint name="$(arg prefix)joint_5" value="0" />
-        <joint name="$(arg prefix)joint_6" value="-0.87" />
-        <joint name="$(arg prefix)joint_7" value="1.57" />
+        <joint name="joint_1" value="0"/>
+        <joint name="joint_2" value="0.2619"/>
+        <joint name="joint_3" value="3.14159"/>
+        <joint name="joint_4" value="-2.269"/>
+        <joint name="joint_5" value="0"/>
+        <joint name="joint_6" value="0.9598"/>
+        <joint name="joint_7" value="1.5708"/>
     </group_state>
     <group_state name="vertical" group="arm">
-        <joint name="$(arg prefix)joint_1" value="0" />
-        <joint name="$(arg prefix)joint_2" value="0" />
-        <joint name="$(arg prefix)joint_3" value="0" />
-        <joint name="$(arg prefix)joint_4" value="0" />
-        <joint name="$(arg prefix)joint_5" value="0" />
-        <joint name="$(arg prefix)joint_6" value="0" />
-        <joint name="$(arg prefix)joint_7" value="0" />
+        <joint name="joint_1" value="0"/>
+        <joint name="joint_2" value="0"/>
+        <joint name="joint_3" value="0"/>
+        <joint name="joint_4" value="0"/>
+        <joint name="joint_5" value="0"/>
+        <joint name="joint_6" value="0"/>
+        <joint name="joint_7" value="0"/>
     </group_state>
+    <!--END EFFECTOR: Purpose: Represent information about an end effector.-->
+    <end_effector name="reamer" parent_link="bracelet_link" group="reamer"/>
+    <!--VIRTUAL JOINT: Purpose: this element defines a virtual joint between a robot link and an external frame of reference (considered fixed with respect to the robot)-->
+    <virtual_joint name="world_frame" type="fixed" parent_frame="world" child_link="base_link"/>
     <!--DISABLE COLLISIONS: By default it is assumed that any link of the robot could potentially come into collision with any other link in the robot. This tag disables collision checking between a specified pair of links. -->
-    <disable_collisions link1="$(arg prefix)bracelet_link" link2="$(arg prefix)forearm_link" reason="Never" />
-    <disable_collisions link1="$(arg prefix)bracelet_link" link2="$(arg prefix)spherical_wrist_1_link" reason="Never" />
-    <disable_collisions link1="$(arg prefix)bracelet_link" link2="$(arg prefix)spherical_wrist_2_link" reason="Adjacent" />
-    <disable_collisions link1="$(arg prefix)forearm_link" link2="$(arg prefix)half_arm_1_link" reason="Never" />
-    <disable_collisions link1="$(arg prefix)bracelet_link" link2="$(arg prefix)forearm_link" reason="Never" />
-    <disable_collisions link1="$(arg prefix)bracelet_link" link2="$(arg prefix)spherical_wrist_1_link" reason="Never" />
-    <disable_collisions link1="$(arg prefix)bracelet_link" link2="$(arg prefix)spherical_wrist_2_link" reason="Adjacent" />
-    <disable_collisions link1="$(arg prefix)forearm_link" link2="$(arg prefix)half_arm_1_link" reason="Never" />
-    <disable_collisions link1="$(arg prefix)forearm_link" link2="$(arg prefix)half_arm_2_link" reason="Adjacent" />
-    <disable_collisions link1="$(arg prefix)forearm_link" link2="$(arg prefix)shoulder_link" reason="Never" />
-    <disable_collisions link1="$(arg prefix)forearm_link" link2="$(arg prefix)spherical_wrist_1_link" reason="Adjacent" />
-    <disable_collisions link1="$(arg prefix)forearm_link" link2="$(arg prefix)spherical_wrist_2_link" reason="Never" />
-    <disable_collisions link1="$(arg prefix)forearm_link" link2="$(arg prefix)base_link" reason="Never" />
-    <disable_collisions link1="$(arg prefix)half_arm_1_link" link2="$(arg prefix)half_arm_2_link" reason="Adjacent" />
-    <disable_collisions link1="$(arg prefix)half_arm_1_link" link2="$(arg prefix)shoulder_link" reason="Adjacent" />
-    <disable_collisions link1="$(arg prefix)half_arm_1_link" link2="$(arg prefix)spherical_wrist_1_link" reason="Never" />
-    <disable_collisions link1="$(arg prefix)half_arm_1_link" link2="$(arg prefix)spherical_wrist_2_link" reason="Never" />
-    <disable_collisions link1="$(arg prefix)half_arm_1_link" link2="$(arg prefix)base_link" reason="Never" />
-    <disable_collisions link1="$(arg prefix)half_arm_2_link" link2="$(arg prefix)shoulder_link" reason="Never" />
-    <disable_collisions link1="$(arg prefix)half_arm_2_link" link2="$(arg prefix)spherical_wrist_1_link" reason="Never" />
-    <disable_collisions link1="$(arg prefix)half_arm_2_link" link2="$(arg prefix)spherical_wrist_2_link" reason="Never" />
-    <disable_collisions link1="$(arg prefix)half_arm_2_link" link2="$(arg prefix)base_link" reason="Never" />
-    <disable_collisions link1="$(arg prefix)shoulder_link" link2="$(arg prefix)spherical_wrist_1_link" reason="Never" />
-    <disable_collisions link1="$(arg prefix)shoulder_link" link2="$(arg prefix)spherical_wrist_2_link" reason="Never" />
-    <disable_collisions link1="$(arg prefix)shoulder_link" link2="$(arg prefix)base_link" reason="Adjacent" />
-    <disable_collisions link1="$(arg prefix)spherical_wrist_1_link" link2="$(arg prefix)spherical_wrist_2_link" reason="Adjacent" />
+    <disable_collisions link1="base_link" link2="forearm_link" reason="Never"/>
+    <disable_collisions link1="base_link" link2="half_arm_1_link" reason="Never"/>
+    <disable_collisions link1="base_link" link2="half_arm_2_link" reason="Never"/>
+    <disable_collisions link1="base_link" link2="shoulder_link" reason="Adjacent"/>
+    <disable_collisions link1="bracelet_link" link2="ee_adapter_link" reason="Adjacent"/>
+    <disable_collisions link1="bracelet_link" link2="forearm_link" reason="Never"/>
+    <disable_collisions link1="bracelet_link" link2="spherical_wrist_1_link" reason="Never"/>
+    <disable_collisions link1="bracelet_link" link2="spherical_wrist_2_link" reason="Adjacent"/>
+    <disable_collisions link1="ee_adapter_link" link2="forearm_link" reason="Never"/>
+    <disable_collisions link1="ee_adapter_link" link2="spherical_wrist_1_link" reason="Never"/>
+    <disable_collisions link1="ee_adapter_link" link2="spherical_wrist_2_link" reason="Never"/>
+    <disable_collisions link1="forearm_link" link2="half_arm_1_link" reason="Never"/>
+    <disable_collisions link1="forearm_link" link2="half_arm_2_link" reason="Adjacent"/>
+    <disable_collisions link1="forearm_link" link2="shoulder_link" reason="Never"/>
+    <disable_collisions link1="forearm_link" link2="spherical_wrist_1_link" reason="Adjacent"/>
+    <disable_collisions link1="forearm_link" link2="spherical_wrist_2_link" reason="Never"/>
+    <disable_collisions link1="half_arm_1_link" link2="half_arm_2_link" reason="Adjacent"/>
+    <disable_collisions link1="half_arm_1_link" link2="shoulder_link" reason="Adjacent"/>
+    <disable_collisions link1="half_arm_1_link" link2="spherical_wrist_1_link" reason="Never"/>
+    <disable_collisions link1="half_arm_2_link" link2="shoulder_link" reason="Never"/>
+    <disable_collisions link1="half_arm_2_link" link2="spherical_wrist_1_link" reason="Never"/>
+    <disable_collisions link1="half_arm_2_link" link2="spherical_wrist_2_link" reason="Never"/>
+    <disable_collisions link1="shoulder_link" link2="spherical_wrist_1_link" reason="Never"/>
+    <disable_collisions link1="spherical_wrist_1_link" link2="spherical_wrist_2_link" reason="Adjacent"/>
 </robot>

Commit message: Finished wrench controller, and updated mass of reamer in urdf

File: kortex_description/arms/gen3/7dof/urdf/gen3_macro.xacro (robot description, xacro)
@@ -301,5 +301,5 @@
       <inertial>
         <origin xyz="-9.3E-05 0.000132 -0.022905" rpy="0 0 0" />
-        <mass value="0.130" />
+        <mass value="1.100" />
         <inertia ixx="0.000214" ixy="0" ixz="1E-06" iyy="0.000223" iyz="-2E-06" izz="0.00024" />
       </inertial>

Commit message: Updating wrench controller and motion planner

File: kortex_description/arms/gen3/7dof/urdf/gen3_macro.xacro (robot description, xacro)
@@ -419,5 +419,5 @@
       name="${prefix}end_effector"
       type="fixed">
-      <origin xyz="0 0 0.29990848" rpy="0 0 0" />
+      <origin xyz="0 0 0" rpy="0 0 0" />
       <parent
         link="${prefix}ee_adapter_link" />
@@ -427,4 +427,5 @@
         xyz="0 0 0" />
     </joint>
+ <!-- 0.29990848 -->
      <!-- <joint
       name="${prefix}reamer_link"

File: kortex_description/robots/kortex_table.xacro (robot description, xacro)
@@ -82,5 +82,5 @@
             <link name="${prefix}tool_frame"/>
             <joint name="${prefix}tool_frame_joint" type="fixed">
-                <origin xyz="0 0 0" rpy="0 0 0" />
+                <origin xyz="0 0 0.29990848" rpy="0 0 0" />
                 <parent link="${prefix}${last_arm_link}" />
                 <child link="${prefix}tool_frame" />

File: kortex_move_it_config/gen3_move_it_config/config/7dof/gen3.srdf.xacro (robot description, xacro)
@@ -19,10 +19,13 @@
         <joint name="joint_6"/>
         <joint name="joint_7"/>
-    </group>
-    <group name="reamer">
         <joint name="ee_joint"/>
         <joint name="end_effector"/>
         <joint name="tool_frame_joint"/>
     </group>
+    <!-- <group name="reamer">
+        <joint name="ee_joint"/>
+        <joint name="end_effector"/>
+        <joint name="tool_frame_joint"/>
+    </group> -->
     <!--GROUP STATES: Purpose: Define a named state for a particular group, in terms of joint values. This is useful to define states like 'folded arms'-->
     <group_state name="home" group="arm">
@@ -45,5 +48,5 @@
     </group_state>
     <!--END EFFECTOR: Purpose: Represent information about an end effector.-->
-    <end_effector name="reamer" parent_link="bracelet_link" group="reamer"/>
+    <!-- <end_effector name="reamer" parent_link="bracelet_link" group="reamer"/> -->
     <!--VIRTUAL JOINT: Purpose: this element defines a virtual joint between a robot link and an external frame of reference (considered fixed with respect to the robot)-->
     <virtual_joint name="world_frame" type="fixed" parent_frame="world" child_link="base_link"/>

File: kortex_move_it_config/gen3_move_it_config/config/7dof/gen3.srdf_new.xacro (robot description, xacro)
@@ -19,6 +19,4 @@
         <joint name="joint_6"/>
         <joint name="joint_7"/>
-    </group>
-    <group name="reamer">
         <joint name="ee_joint"/>
         <joint name="end_effector"/>
@@ -26,9 +24,22 @@
     </group>
     <!--GROUP STATES: Purpose: Define a named state for a particular group, in terms of joint values. This is useful to define states like 'folded arms'-->
-    <group_state name="home" group="arm"/>
-    <group_state name="retract" group="arm"/>
-    <group_state name="vertical" group="arm"/>
-    <!--END EFFECTOR: Purpose: Represent information about an end effector.-->
-    <end_effector name="reamer" parent_link="bracelet_link" group="reamer"/>
+    <group_state name="home" group="arm">
+        <joint name="joint_1" value="0"/>
+        <joint name="joint_2" value="0.2619"/>
+        <joint name="joint_3" value="3.14159"/>
+        <joint name="joint_4" value="-2.269"/>
+        <joint name="joint_5" value="0"/>
+        <joint name="joint_6" value="0.9598"/>
+        <joint name="joint_7" value="1.5708"/>
+    </group_state>
+    <group_state name="vertical" group="arm">
+        <joint name="joint_1" value="0"/>
+        <joint name="joint_2" value="0"/>
+        <joint name="joint_3" value="0"/>
+        <joint name="joint_4" value="0"/>
+        <joint name="joint_5" value="0"/>
+        <joint name="joint_6" value="0"/>
+        <joint name="joint_7" value="0"/>
+    </group_state>
     <!--VIRTUAL JOINT: Purpose: this element defines a virtual joint between a robot link and an external frame of reference (considered fixed with respect to the robot)-->
     <virtual_joint name="world_frame" type="fixed" parent_frame="world" child_link="base_link"/>

Commit message: End of spring semester

File: kortex_description/arms/gen3/7dof/urdf/gen3_macro.xacro (robot description, xacro)
@@ -305,16 +305,16 @@
       </inertial>
       <visual>
-        <origin xyz="-0.04 -0.04 0" rpy="0 0 0" />
-        <geometry>
-          <mesh filename="package://kortex_description/arms/gen3/${dof}dof/meshes/ReamerAssemblyCombine.stl" scale="0.001 0.001 0.001"/>
-        </geometry>
-        <material name="">
-          <color rgba="0.75294 0.75294 0.75294 1" />
-        </material>
-      </visual>
-      <collision>
-        <origin xyz="-0.04 -0.04 0" rpy="0 0 0" />
-        <geometry>
-          <mesh filename="package://kortex_description/arms/gen3/${dof}dof/meshes/ReamerAssemblyCombine.stl" scale="0.001 0.001 0.001"/>
+        <origin xyz="0 0 0" rpy="0 0 0" />
+        <geometry>
+          <mesh filename="package://kortex_description/arms/gen3/${dof}dof/meshes/ReamerAssemblyCombine.stl"/>
+        </geometry>
+        <material name="">
+          <color rgba="0.75294 0.75294 0.75294 1" />
+        </material>
+      </visual>
+      <collision>
+        <origin xyz="0 0 0" rpy="0 0 0" />
+        <geometry>
+          <mesh filename="package://kortex_description/arms/gen3/${dof}dof/meshes/ReamerAssemblyCombine.stl"/>
         </geometry>
       </collision>

Commit message: Got basic task prioritization working with 5dof task. Still some bugs to fix such as it freaks out when restarting from random point.

File: kortex_description/arms/gen3/7dof/urdf/gen3_macro.xacro (robot description, xacro)
@@ -94,5 +94,5 @@
       <axis
         xyz="0 0 1" />
-      <limit lower="-2.41" upper="2.41" effort="39" velocity="1.3963" />
+      <limit lower="-2.15" upper="2.15" effort="39" velocity="1.3963" />
     </joint>
     <link name="${prefix}half_arm_2_link">

Commit message: Calibrated the of the arm base

File: kortex_description/arms/gen3/7dof/urdf/gen3_macro.xacro (robot description, xacro)
@@ -331,5 +331,4 @@
     <link name="${prefix}ee_marker_frame"/>
     <joint name="${prefix}ee_marker_frame_joint" type="fixed">
-        <!-- <origin xyz="0.034 0.0457193 0.14223149" rpy="0 -1.570796327 0" /> -->
         <origin xyz="0.042 0.0417193 0.14523149" rpy="0 -1.570796327 0" />
         <!-- <origin xyz="0 0.01025305 0.17316221" rpy="0 -1.570796327 0" /> -->
@@ -340,5 +339,4 @@
     <link name="${prefix}ee_reamer_hole"/>
     <joint name="${prefix}ee_reamer_hole_joint" type="fixed">
-        <!-- <origin xyz="0.03093072 -0.02746625 0.034" rpy="-1.570796327 -1.570796327 0.7853981635" /> -->
         <origin xyz="0.02793072 -0.03146625 0.042" rpy="-1.570796327 -1.570796327 0.7853981635" />
         <parent link="${prefix}ee_marker_frame" />
