Commit message: sundaram commits

File: kortex_description/robots/kortex_table.xacro (robot description, xacro)
@@ -52,5 +52,5 @@
                 <parent link="table" />
                 <child link = "pelvis_link" />
-                <origin xyz="0 0.3 0.01" rpy="-1.57 0 0" />
+                <origin xyz="0.5 0.3 0.01" rpy="0.5 0 2.0" />
                 <limit lower="-3.1416" upper="3.1416" effort="10" velocity="3"/>
                 <axis xyz="0 1 0"/>

Commit message: planning and controls integrated

File: kortex_description/robots/kortex_table.xacro (robot description, xacro)
@@ -80,9 +80,16 @@
         <!-- If no gripper, define tool frame here -->
         <xacro:if value="${not gripper}">
+            <link name="${prefix}tool_tip_frame"/>
+            <joint name="${prefix}tool_tip_frame_joint" type="fixed">
+                <origin xyz="0 0 0.32290848" rpy="0 0 0" />
+                <parent link="${prefix}${last_arm_link}" />
+                <child link="${prefix}tool_tip_frame" />
+                <axis xyz="0 0 0" />
+            </joint>
             <link name="${prefix}tool_frame"/>
             <joint name="${prefix}tool_frame_joint" type="fixed">
-                <origin xyz="0 0 0.29990848" rpy="0 0 0" />
-                <parent link="${prefix}${last_arm_link}" />
-                <child link="${prefix}tool_frame" />
+                <origin xyz="0 0 -0.023" rpy="0 0 0" />
+                <parent link="${prefix}tool_tip_frame" />
+                <child link="${prefix}tool_frame"/>
                 <axis xyz="0 0 0" />
             </joint>

File: kortex_move_it_config/gen3_move_it_config/config/7dof/gen3.srdf.xacro (robot description, xacro)
@@ -21,5 +21,5 @@
         <joint name="ee_joint"/>
         <joint name="end_effector"/>
-        <joint name="tool_frame_joint"/>
+        <joint name="tool_tip_frame_joint"/>
     </group>
     <!-- <group name="reamer">

Commit message: Finished online calibration v1

File: kortex_description/robots/kortex_table.xacro (robot description, xacro)
@@ -22,5 +22,5 @@
             <link name="table">
                 <visual>
-                    <origin xyz="0 0 0.01" rpy="1.5708 0 0" />
+                    <origin xyz="0 0 0.02" rpy="1.5708 0 0" />
                     <geometry>
                         <mesh filename="package://kortex_description/meshes/environment/Table_v2.STL"/>
@@ -28,5 +28,5 @@
                 </visual>
                 <collision>
-                    <origin xyz="0 0 0" rpy="1.5708 0 0" />
+                    <origin xyz="0 0 0.02" rpy="1.5708 0 0" />
                     <geometry>
                         <mesh filename="package://kortex_description/meshes/environment/Table_v2.STL"/>
