Commit message: IK Controller v1

File: kortex_control/arm_description/robot_model.xacro (robot description, xacro)
@@ -8,5 +8,5 @@
     <xacro:arg name="sim" default="false" />
     <xacro:arg name="prefix" default="" />
-    <xacro:include filename="$(find kortex_description)/robots/kortex_robot.xacro" />
+    <xacro:include filename="$(find kortex_description)/arms/$(arg arm)/$(arg dof)dof/urdf/$(arg arm)_macro.xacro" />
     <link name="world" />
     <joint name="world_to_root" type="fixed">
@@ -15,4 +15,21 @@
         <origin xyz="0 0 0" rpy="0 0 0" />
     </joint>
-    <xacro:load_robot arm="$(arg arm)" gripper="$(arg gripper)" dof="$(arg dof)" vision="$(arg vision)" sim="$(arg sim)" prefix="$(arg prefix)" />
+    <xacro:load_arm parent="" dof="$(arg dof)" vision="$(arg vision)" prefix="$(arg prefix)">
+        <origin xyz="0 0 0" rpy="0 0 0"/>
+    </xacro:load_arm>
+    <!-- TODO: If the following is changed, need to change also in kortex_table and in kortex_robot xacros -->
+    <link name="$(arg prefix)tool_tip_frame"/>
+    <joint name="$(arg prefix)tool_tip_frame_joint" type="fixed">
+        <origin xyz="0 0 0.32290848" rpy="0 0 0" />
+        <parent link="$(arg prefix)${last_arm_link}" />
+        <child link="$(arg prefix)tool_tip_frame" />
+        <axis xyz="0 0 0" />
+    </joint>
+    <link name="$(arg prefix)tool_frame"/>
+    <joint name="$(arg prefix)tool_frame_joint" type="fixed">
+        <origin xyz="0 0 -0.023" rpy="0 0 0" />
+        <parent link="$(arg prefix)tool_tip_frame" />
+        <child link="$(arg prefix)tool_frame"/>
+        <axis xyz="0 0 0" />
+    </joint>
 </robot>

File: kortex_description/robots/kortex_robot.xacro (robot description, xacro)
@@ -35,4 +35,5 @@
         </xacro:unless>
         <!-- If no gripper, define tool frame here -->
+        <!-- TODO: If the following is changed, need to change also in kortex_table and in robot_model (Kortex Control) -->
         <xacro:if value="${not gripper}">
             <link name="${prefix}tool_frame"/>

File: kortex_description/robots/kortex_table.xacro (robot description, xacro)
@@ -79,4 +79,5 @@
         </xacro:unless>
         <!-- If no gripper, define tool frame here -->
+        <!-- TODO: If the following is changed, need to change also in kortex_robot and in robot_model (Kortex Control) -->
         <xacro:if value="${not gripper}">
             <link name="${prefix}tool_tip_frame"/>

Commit message: Fixed bugs and now working on real arm

File: kortex_control/arm_description/robot_model.xacro (robot description, xacro)
@@ -21,5 +21,5 @@
     <link name="$(arg prefix)tool_tip_frame"/>
     <joint name="$(arg prefix)tool_tip_frame_joint" type="fixed">
-        <origin xyz="0 0 0.32290848" rpy="0 0 0" />
+        <origin xyz="0 0 0.32290848" rpy="3.14159265 0 0" />
         <parent link="$(arg prefix)${last_arm_link}" />
         <child link="$(arg prefix)tool_tip_frame" />
@@ -28,5 +28,5 @@
     <link name="$(arg prefix)tool_frame"/>
     <joint name="$(arg prefix)tool_frame_joint" type="fixed">
-        <origin xyz="0 0 -0.023" rpy="0 0 0" />
+        <origin xyz="0 0 0.023" rpy="0 0 0" />
         <parent link="$(arg prefix)tool_tip_frame" />
         <child link="$(arg prefix)tool_frame"/>

File: kortex_description/robots/kortex_table.xacro (robot description, xacro)
@@ -83,5 +83,5 @@
             <link name="${prefix}tool_tip_frame"/>
             <joint name="${prefix}tool_tip_frame_joint" type="fixed">
-                <origin xyz="0 0 0.32290848" rpy="0 0 0" />
+                <origin xyz="0 0 0.32290848" rpy="3.14159265 0 0" />
                 <parent link="${prefix}${last_arm_link}" />
                 <child link="${prefix}tool_tip_frame" />
@@ -90,5 +90,5 @@
             <link name="${prefix}tool_frame"/>
             <joint name="${prefix}tool_frame_joint" type="fixed">
-                <origin xyz="0 0 -0.023" rpy="0 0 0" />
+                <origin xyz="0 0 0.023" rpy="0 0 0" />
                 <parent link="${prefix}tool_tip_frame" />
                 <child link="${prefix}tool_frame"/>

Commit message: Fixed joint limit bugs and Added camera alignment task with task prioritization

File: kortex_control/arm_description/robot_model.xacro (robot description, xacro)
@@ -19,8 +19,15 @@
     </xacro:load_arm>
     <!-- TODO: If the following is changed, need to change also in kortex_table and in kortex_robot xacros -->
+    <link name="$(arg prefix)ee_marker_frame"/>
+    <joint name="$(arg prefix)ee_marker_frame_joint" type="fixed">
+        <origin xyz="0 0 0.16" rpy="1.5708 0 0" />
+        <parent link="$(arg prefix)${last_arm_link}" />
+        <child link="$(arg prefix)ee_marker_frame" />
+        <axis xyz="0 0 0" />
+    </joint>
     <link name="$(arg prefix)tool_tip_frame"/>
     <joint name="$(arg prefix)tool_tip_frame_joint" type="fixed">
-        <origin xyz="0 0 0.32290848" rpy="3.14159265 0 0" />
-        <parent link="$(arg prefix)${last_arm_link}" />
+        <origin xyz="0 0.16290848 0" rpy="1.5708 0 0" />
+        <parent link="$(arg prefix)ee_marker_frame" />
         <child link="$(arg prefix)tool_tip_frame" />
         <axis xyz="0 0 0" />

File: kortex_description/arms/gen3/7dof/urdf/gen3_macro.xacro (robot description, xacro)
@@ -94,5 +94,5 @@
       <axis
         xyz="0 0 1" />
-      <limit lower="-2.15" upper="2.15" effort="39" velocity="1.3963" />
+      <limit lower="-2.05" upper="2.05" effort="39" velocity="1.3963" />
     </joint>
     <link name="${prefix}half_arm_2_link">

File: kortex_description/robots/kortex_table.xacro (robot description, xacro)
@@ -81,8 +81,15 @@
         <!-- TODO: If the following is changed, need to change also in kortex_robot and in robot_model (Kortex Control) -->
         <xacro:if value="${not gripper}">
+            <link name="${prefix}ee_marker_frame"/>
+            <joint name="${prefix}ee_marker_frame_joint" type="fixed">
+                <origin xyz="0 0 0.16" rpy="1.5708 0 0" />
+                <parent link="${prefix}${last_arm_link}" />
+                <child link="${prefix}ee_marker_frame" />
+                <axis xyz="0 0 0" />
+            </joint>
             <link name="${prefix}tool_tip_frame"/>
             <joint name="${prefix}tool_tip_frame_joint" type="fixed">
-                <origin xyz="0 0 0.32290848" rpy="3.14159265 0 0" />
-                <parent link="${prefix}${last_arm_link}" />
+                <origin xyz="0 0.16290848 0" rpy="1.5708 0 0" />
+                <parent link="${prefix}ee_marker_frame" />
                 <child link="${prefix}tool_tip_frame" />
                 <axis xyz="0 0 0" />

Commit message: Updated urdf

File: kortex_control/arm_description/robot_model.xacro (robot description, xacro)
@@ -21,21 +21,21 @@
     <link name="$(arg prefix)ee_marker_frame"/>
     <joint name="$(arg prefix)ee_marker_frame_joint" type="fixed">
-        <origin xyz="0 0 0.16" rpy="1.5708 0 0" />
+        <origin xyz="0 0 0" rpy="-1.5708 0 0" />
         <parent link="$(arg prefix)${last_arm_link}" />
         <child link="$(arg prefix)ee_marker_frame" />
         <axis xyz="0 0 0" />
     </joint>
+    <link name="$(arg prefix)tool_frame"/>
+    <joint name="$(arg prefix)tool_frame_joint" type="fixed">
+        <origin xyz="-0.008480 -0.191619 0 " rpy="-1.5708 0 -0.7854" />
+        <parent link="$(arg prefix)ee_marker_frame" />
+        <child link="$(arg prefix)tool_frame" />
+        <axis xyz="0 0 0" />
+    </joint>
     <link name="$(arg prefix)tool_tip_frame"/>
     <joint name="$(arg prefix)tool_tip_frame_joint" type="fixed">
-        <origin xyz="0 0.16290848 0" rpy="1.5708 0 0" />
-        <parent link="$(arg prefix)ee_marker_frame" />
-        <child link="$(arg prefix)tool_tip_frame" />
-        <axis xyz="0 0 0" />
-    </joint>
-    <link name="$(arg prefix)tool_frame"/>
-    <joint name="$(arg prefix)tool_frame_joint" type="fixed">
-        <origin xyz="0 0 0.023" rpy="0 0 0" />
-        <parent link="$(arg prefix)tool_tip_frame" />
-        <child link="$(arg prefix)tool_frame"/>
+        <origin xyz="0 0 -0.023" rpy="0 0 0" />
+        <parent link="$(arg prefix)tool_frame" />
+        <child link="$(arg prefix)tool_tip_frame"/>
         <axis xyz="0 0 0" />
     </joint>

File: kortex_control/arm_description/test.urdf (robot description, URDF)
Before this commit: robot gen3, 13 links, 12 joints
Links:
- added link ee_marker_frame
- link ee_adapter_link: geometry collision mesh filename=package://kortex_description/arms/gen3/7dof/meshes/EE_V1_co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; visual mesh filename=package://kortex_description/arms/gen3/7dof/meshes/EE_V1_co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
Joints:
- added joint ee_marker_frame_joint: type fixed, parent end_effector_link, child ee_marker_frame, origin xyz=0 0 0 rpy=-1.5708 0 0, axis 0 0 0
- joint ee_joint: origin xyz=0 0 -0.0615250000000001 rpy=3.14159265358979 1.09937075168372E-32 0 -> xyz=0 0 -0.06446 rpy=3.14159265358979 0 1.5708
- joint joint_2: limit lower=-2.41 upper=2.41 effort=39 velocity=1.3963 -> lower=-2.05 upper=2.05 effort=39 velocity=1.3963
- joint tool_frame_joint: origin xyz=0 0 -0.023 rpy=0 0 0 -> xyz=-0.008480 -0.191619 0  rpy=-1.5708 0 -0.7854; parent tool_tip_frame -> ee_marker_frame
- joint tool_tip_frame_joint: origin xyz=0 0 0.32290848 rpy=0 0 0 -> xyz=0 0 -0.023 rpy=0 0 0; parent end_effector_link -> tool_frame

File: kortex_description/arms/gen3/7dof/urdf/gen3_macro.xacro (robot description, xacro)
@@ -298,5 +298,5 @@
         velocity="1.2218" />
     </joint>
-    <link name="${prefix}ee_adapter_link">
+    <!-- <link name="${prefix}ee_adapter_link">
       <inertial>
         <origin xyz="-9.3E-05 0.000132 -0.022905" rpy="0 0 0" />
@@ -319,7 +319,38 @@
         </geometry>
       </collision>
+    </link> -->
+    <!-- <joint name="${prefix}ee_joint" type="fixed">
+      <origin xyz="0 0 -0.0615250000000001" rpy="3.14159265358979 1.09937075168372E-32 0" />
+      <parent
+        link="${prefix}bracelet_link" />
+      <child
+        link="${prefix}ee_adapter_link" />
+      <axis
+        xyz="0 0 0" />
+    </joint> -->
+    <link name="${prefix}ee_adapter_link">
+      <inertial>
+        <origin xyz="-9.3E-05 0.000132 -0.022905" rpy="0 0 0" />
+        <mass value="1.100" />
+        <inertia ixx="0.000214" ixy="0" ixz="1E-06" iyy="0.000223" iyz="-2E-06" izz="0.00024" />
+      </inertial>
+      <visual>
+        <origin xyz="0 0 0" rpy="0 0 0" />
+        <geometry>
+          <mesh filename="package://kortex_description/arms/gen3/${dof}dof/meshes/EE_V1_compressed.stl"/>
+        </geometry>
+        <material name="">
+          <color rgba="0.75294 0.75294 0.75294 1" />
+        </material>
+      </visual>
+      <collision>
+        <origin xyz="0 0 0" rpy="0 0 0" />
+        <geometry>
+          <mesh filename="package://kortex_description/arms/gen3/${dof}dof/meshes/EE_V1_compressed.stl"/>
+        </geometry>
+      </collision>
     </link>
     <joint name="${prefix}ee_joint" type="fixed">
-      <origin xyz="0 0 -0.0615250000000001" rpy="3.14159265358979 1.09937075168372E-32 0" />
+      <origin xyz="0 0 -0.06446" rpy="3.14159265358979 0 1.5708" />
       <parent
         link="${prefix}bracelet_link" />

File: kortex_description/robots/kortex_table.xacro (robot description, xacro)
@@ -83,12 +83,26 @@
             <link name="${prefix}ee_marker_frame"/>
             <joint name="${prefix}ee_marker_frame_joint" type="fixed">
-                <origin xyz="0 0 0.16" rpy="1.5708 0 0" />
+                <origin xyz="0 0 0" rpy="-1.5708 0 0" />
                 <parent link="${prefix}${last_arm_link}" />
                 <child link="${prefix}ee_marker_frame" />
                 <axis xyz="0 0 0" />
             </joint>
+            <link name="${prefix}tool_frame"/>
+            <joint name="${prefix}tool_frame_joint" type="fixed">
+                <origin xyz="-0.008480 -0.191619 0 " rpy="-1.5708 0 -0.7854" />
+                <parent link="${prefix}ee_marker_frame" />
+                <child link="${prefix}tool_frame" />
+                <axis xyz="0 0 0" />
+            </joint>
             <link name="${prefix}tool_tip_frame"/>
             <joint name="${prefix}tool_tip_frame_joint" type="fixed">
-                <origin xyz="0 0.16290848 0" rpy="1.5708 0 0" />
+                <origin xyz="0 0 -0.023" rpy="0 0 0" />
+                <parent link="${prefix}tool_frame" />
+                <child link="${prefix}tool_tip_frame"/>
+                <axis xyz="0 0 0" />
+            </joint>
+            <!-- <link name="${prefix}tool_tip_frame"/>
+            <joint name="${prefix}tool_tip_frame_joint" type="fixed">
+                <origin xyz="0 -0.16290848 0" rpy="-1.5708 0 0" />
                 <parent link="${prefix}ee_marker_frame" />
                 <child link="${prefix}tool_tip_frame" />
@@ -101,5 +115,5 @@
                 <child link="${prefix}tool_frame"/>
                 <axis xyz="0 0 0" />
-            </joint>
+            </joint> -->
         </xacro:if>
         <!-- Load the Gazebo transmissions and gazebo_ros_control plugin -->
