Commit message: Updated urdf and modified arm controls to use tool frame tip (untested)

File: kortex_control/arm_description/robot_model.xacro (robot description, xacro)
@@ -19,22 +19,55 @@
     </xacro:load_arm>
     <!-- TODO: If the following is changed, need to change also in kortex_table and in kortex_robot xacros -->
-    <link name="$(arg prefix)ee_marker_frame"/>
-    <joint name="$(arg prefix)ee_marker_frame_joint" type="fixed">
-        <origin xyz="0 0 0" rpy="-1.5708 0 0" />
+    <link name="$(arg prefix)tool_frame">
+        <visual>
+            <origin xyz="0 0 0" rpy="0 0 0" />
+            <geometry>
+            <mesh filename="package://kortex_description/arms/gen3/$(arg dof)dof/meshes/ReamerHead.STL"/>
+            </geometry>
+            <material name="">
+            <color rgba="0.75294 0.75294 0.75294 1" />
+            </material>
+        </visual>
+        <collision>
+            <origin xyz="0 0 0" rpy="0 0 0" />
+            <geometry>
+            <mesh filename="package://kortex_description/arms/gen3/$(arg dof)dof/meshes/ReamerHead.STL"/>
+            </geometry>
+        </collision>
+    </link>
+    <joint name="$(arg prefix)tool_frame_joint" type="fixed">
+        <origin xyz="0 0 -0.0915" rpy="0 0 0" />
         <parent link="$(arg prefix)${last_arm_link}" />
-        <child link="$(arg prefix)ee_marker_frame" />
+        <child link="$(arg prefix)tool_frame" />
         <axis xyz="0 0 0" />
+        <!-- <limit lower="-0.07" upper="0" effort="200" velocity="40" /> -->
     </joint>
-    <link name="$(arg prefix)tool_frame"/>
-    <joint name="$(arg prefix)tool_frame_joint" type="fixed">
-        <origin xyz="-0.008480 -0.191619 0 " rpy="-1.5708 0 -0.7854" />
-        <parent link="$(arg prefix)ee_marker_frame" />
-        <child link="$(arg prefix)tool_frame" />
+    <link name="$(arg prefix)reamer_head">
+        <visual>
+            <origin xyz="0 0 0" rpy="0 0 0" />
+            <geometry>
+            <mesh filename="package://kortex_description/arms/gen3/$(arg dof)dof/meshes/ReamingHead_56MM.STL"/>
+            </geometry>
+            <material name="">
+            <color rgba="0.75294 0.75294 0.75294 1" />
+            </material>
+        </visual>
+        <collision>
+            <origin xyz="0 0 0" rpy="0 0 0" />
+            <geometry>
+            <mesh filename="package://kortex_description/arms/gen3/$(arg dof)dof/meshes/ReamingHead_56MM.STL"/>
+            </geometry>
+        </collision>
+    </link>
+    <joint name="$(arg prefix)reamer_head_joint" type="fixed">
+        <origin xyz="0 0 0" rpy="0 0 0" />
+        <parent link="$(arg prefix)tool_frame" />
+        <child link="$(arg prefix)reamer_head" />
         <axis xyz="0 0 0" />
     </joint>
     <link name="$(arg prefix)tool_tip_frame"/>
     <joint name="$(arg prefix)tool_tip_frame_joint" type="fixed">
-        <origin xyz="0 0 -0.023" rpy="0 0 0" />
-        <parent link="$(arg prefix)tool_frame" />
+        <origin xyz="0 0 -0.028" rpy="0 0 0" />
+        <parent link="$(arg prefix)reamer_head" />
         <child link="$(arg prefix)tool_tip_frame"/>
         <axis xyz="0 0 0" />

File: kortex_control/arm_description/test.urdf (robot description, URDF)
Before this commit: robot gen3, 14 links, 13 joints
Links:
- added link ee_reamer_hole
- added link reamer_head; collision mesh filename=package://kortex_description/arms/gen3/7dof/meshes/ReamingH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; visual mesh filename=package://kortex_description/arms/gen3/7dof/meshes/ReamingH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
- link ee_adapter_link: geometry collision mesh filename=package://kortex_description/arms/gen3/7dof/meshes/EE_V1.stl; visual mesh filename=package://kortex_description/arms/gen3/7dof/meshes/EE_V1.stl
- link tool_frame: geometry collision mesh filename=package://kortex_description/arms/gen3/7dof/meshes/ReamerHe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; visual mesh filename=package://kortex_description/arms/gen3/7dof/meshes/ReamerHe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
Joints:
- added joint ee_reamer_hole_joint: type fixed, parent ee_marker_frame, child ee_reamer_hole, origin xyz=0.02793072 -0.03146625 0.042 rpy=-1.570796327 -1.570796327 0.7853981635, axis 0 0 0
- added joint reamer_head_joint: type fixed, parent tool_frame, child reamer_head, origin xyz=0 0 0 rpy=0 0 0, axis 0 0 0
- joint ee_joint: origin xyz=0 0 -0.06446 rpy=3.14159265358979 0 1.5708 -> xyz=0 0 -0.06446 rpy=3.14159265358979 0 3.14159265358979
- joint ee_marker_frame_joint: origin xyz=0 0 0 rpy=-1.5708 0 0 -> xyz=0.042 0.0417193 0.14523149 rpy=0 -1.570796327 0; parent end_effector_link -> ee_adapter_link
- joint end_effector: parent ee_adapter_link -> ee_reamer_hole
- joint tool_frame_joint: origin xyz=-0.008480 -0.191619 0  rpy=-1.5708 0 -0.7854 -> xyz=0 0 -0.0915 rpy=0 0 0; parent ee_marker_frame -> end_effector_link
- joint tool_tip_frame_joint: origin xyz=0 0 -0.023 rpy=0 0 0 -> xyz=0 0 -0.028 rpy=0 0 0; parent tool_frame -> reamer_head

File: kortex_description/arms/gen3/7dof/urdf/gen3_macro.xacro (robot description, xacro)
@@ -298,5 +298,5 @@
         velocity="1.2218" />
     </joint>
-    <!-- <link name="${prefix}ee_adapter_link">
+    <link name="${prefix}ee_adapter_link">
       <inertial>
         <origin xyz="-9.3E-05 0.000132 -0.022905" rpy="0 0 0" />
@@ -307,19 +307,19 @@
         <origin xyz="0 0 0" rpy="0 0 0" />
         <geometry>
-          <mesh filename="package://kortex_description/arms/gen3/${dof}dof/meshes/ReamerAssemblyCombine.stl"/>
-        </geometry>
-        <material name="">
-          <color rgba="0.75294 0.75294 0.75294 1" />
-        </material>
-      </visual>
-      <collision>
-        <origin xyz="0 0 0" rpy="0 0 0" />
-        <geometry>
-          <mesh filename="package://kortex_description/arms/gen3/${dof}dof/meshes/ReamerAssemblyCombine.stl"/>
-        </geometry>
-      </collision>
-    </link> -->
-    <!-- <joint name="${prefix}ee_joint" type="fixed">
-      <origin xyz="0 0 -0.0615250000000001" rpy="3.14159265358979 1.09937075168372E-32 0" />
+          <mesh filename="package://kortex_description/arms/gen3/${dof}dof/meshes/EE_V1.stl"/>
+        </geometry>
+        <material name="">
+          <color rgba="0.75294 0.75294 0.75294 1" />
+        </material>
+      </visual>
+      <collision>
+        <origin xyz="0 0 0" rpy="0 0 0" />
+        <geometry>
+          <mesh filename="package://kortex_description/arms/gen3/${dof}dof/meshes/EE_V1.stl"/>
+        </geometry>
+      </collision>
+    </link>
+    <joint name="${prefix}ee_joint" type="fixed">
+      <origin xyz="0 0 -0.06446" rpy="3.14159265358979 0 3.14159265358979" />
       <parent
         link="${prefix}bracelet_link" />
@@ -328,122 +328,20 @@
       <axis
         xyz="0 0 0" />
-    </joint> -->
-    <link name="${prefix}ee_adapter_link">
-      <inertial>
-        <origin xyz="-9.3E-05 0.000132 -0.022905" rpy="0 0 0" />
-        <mass value="1.100" />
-        <inertia ixx="0.000214" ixy="0" ixz="1E-06" iyy="0.000223" iyz="-2E-06" izz="0.00024" />
-      </inertial>
-      <visual>
-        <origin xyz="0 0 0" rpy="0 0 0" />
-        <geometry>
-          <mesh filename="package://kortex_description/arms/gen3/${dof}dof/meshes/EE_V1_compressed.stl"/>
-        </geometry>
-        <material name="">
-          <color rgba="0.75294 0.75294 0.75294 1" />
-        </material>
-      </visual>
-      <collision>
-        <origin xyz="0 0 0" rpy="0 0 0" />
-        <geometry>
-          <mesh filename="package://kortex_description/arms/gen3/${dof}dof/meshes/EE_V1_compressed.stl"/>
-        </geometry>
-      </collision>
-    </link>
-    <joint name="${prefix}ee_joint" type="fixed">
-      <origin xyz="0 0 -0.06446" rpy="3.14159265358979 0 1.5708" />
-      <parent
-        link="${prefix}bracelet_link" />
-      <child
-        link="${prefix}ee_adapter_link" />
-      <axis
-        xyz="0 0 0" />
-    </joint>
-    <!-- <link name="${prefix}ftsensor_link">
-      <inertial>
-        <origin xyz="-9.3E-05 0.000132 -0.022905" rpy="0 0 0" />
-        <mass value="0.310" />
-        <inertia ixx="0.000214" ixy="0" ixz="1E-06" iyy="0.000223" iyz="-2E-06" izz="0.00024" />
-      </inertial>
-      <visual>
-        <origin xyz="-0.04 -0.05 0" rpy="0 0 0" />
-        <geometry>
-          <mesh filename="package://kortex_description/arms/gen3/${dof}dof/meshes/FTSensor.STL" scale="0.001 0.001 0.001"/>
-        </geometry>
-        <material name="">
-          <color rgba="0.75294 0.75294 0.75294 1" />
-        </material>
-      </visual>
-      <collision>
-        <origin xyz="-0.04 -0.05 0" rpy="0 0 0" />
-        <geometry>
-          <mesh filename="package://kortex_description/arms/gen3/${dof}dof/meshes/FTSensor.STL" scale="0.001 0.001 0.001"/>
-        </geometry>
-      </collision>
-    </link>
-    <link name="${prefix}ee_adapter_link">
-      <inertial>
-        <origin xyz="-9.3E-05 0.000132 -0.022905" rpy="0 0 0" />
-        <mass value="0.130" />
-        <inertia ixx="0.000214" ixy="0" ixz="1E-06" iyy="0.000223" iyz="-2E-06" izz="0.00024" />
-      </inertial>
-      <visual>
-        <origin xyz="-0.04 -0.04 0" rpy="0 0 0" />
-        <geometry>
-          <mesh filename="package://kortex_description/arms/gen3/${dof}dof/meshes/FTAdapter.STL" scale="0.001 0.001 0.001"/>
-        </geometry>
-        <material name="">
-          <color rgba="0.75294 0.75294 0.75294 1" />
-        </material>
-      </visual>
-      <collision>
-        <origin xyz="-0.04 -0.04 0" rpy="0 0 0" />
-        <geometry>
-          <mesh filename="package://kortex_description/arms/gen3/${dof}dof/meshes/FTAdapter.STL" scale="0.001 0.001 0.001"/>
-        </geometry>
-      </collision>
-    </link>
-    <link name="${prefix}reamer_link">
-      <inertial>
-        <origin xyz="-9.3E-05 0.000132 -0.022905" rpy="0 0 0" />
-        <mass value="0.130" />
-        <inertia ixx="0.000214" ixy="0" ixz="1E-06" iyy="0.000223" iyz="-2E-06" izz="0.00024" />
-      </inertial>
-      <visual>
-        <origin xyz="-0.04 -0.04 0" rpy="0 0 0" />
-        <geometry>
-          <mesh filename="package://kortex_description/arms/gen3/${dof}dof/meshes/ReamerAssembly.STL" scale="0.001 0.001 0.001"/>
-        </geometry>
-        <material name="">
-          <color rgba="0.75294 0.75294 0.75294 1" />
-        </material>
-      </visual>
-      <collision>
-        <origin xyz="-0.04 -0.04 0" rpy="0 0 0" />
-        <geometry>
-          <mesh filename="package://kortex_description/arms/gen3/${dof}dof/meshes/ReamerAssembly.STL" scale="0.001 0.001 0.001"/>
-        </geometry>
-      </collision>
-    </link>
-    <joint name="${prefix}ft_sensor" type="fixed">
-      <origin xyz="0 0 -0.0615250000000001" rpy="3.14159265358979 1.09937075168372E-32 0" />
-      <parent
-        link="${prefix}bracelet_link" />
-      <child
-        link="${prefix}ee_adapter_link" />
-      <axis
-        xyz="0 0 0" />
-    </joint>
-    <joint
-      name="${prefix}ee_adapter"
-      type="fixed">
-      <origin xyz="0 0 0.075" rpy="0 0 0" />
-      <parent
-        link="${prefix}ee_adapter_link" />
-      <child
-        link="${prefix}ftsensor_link" />
-      <axis
-        xyz="0 0 0" />
-    </joint> -->
+    </joint>
+    <link name="${prefix}ee_marker_frame"/>
+    <joint name="${prefix}ee_marker_frame_joint" type="fixed">
+        <origin xyz="0.042 0.0417193 0.14523149" rpy="0 -1.570796327 0" />
+        <!-- <origin xyz="0 0.01025305 0.17316221" rpy="0 -1.570796327 0" /> -->
+        <parent link="${prefix}ee_adapter_link" />
+        <child link="${prefix}ee_marker_frame" />
+        <axis xyz="0 0 0" />
+    </joint>
+    <link name="${prefix}ee_reamer_hole"/>
+    <joint name="${prefix}ee_reamer_hole_joint" type="fixed">
+        <origin xyz="0.02793072 -0.03146625 0.042" rpy="-1.570796327 -1.570796327 0.7853981635" />
+        <parent link="${prefix}ee_marker_frame" />
+        <child link="${prefix}ee_reamer_hole" />
+        <axis xyz="0 0 0" />
+    </joint>
     <link name="${prefix}end_effector_link" />
     <joint
@@ -452,5 +350,5 @@
       <origin xyz="0 0 0" rpy="0 0 0" />
       <parent
-        link="${prefix}ee_adapter_link" />
+        link="${prefix}ee_reamer_hole" />
       <child
         link="${prefix}end_effector_link" />
@@ -458,60 +356,4 @@
         xyz="0 0 0" />
     </joint>
- <!-- 0.29990848 -->
-     <!-- <joint
-      name="${prefix}reamer_link"
-      type="fixed">
-      <origin xyz="0 0 0.1" rpy="0 0 0" />
-      <parent
-        link="${prefix}ee_adapter_link" />
-      <child
-        link="${prefix}reamer_link" />
-      <axis
-        xyz="0 0 0" />
-    </joint>
-    <link name="${prefix}end_effector_link"/>
-    <joint
-      name="${prefix}end_effector"
-      type="fixed">
-      <origin xyz="0 0 0" rpy="3.14159265358979 1.09937075168372E-32 0" />
-      <parent
-        link="${prefix}reamer_link" />
-      <child
-        link="${prefix}end_effector_link" />
-      <axis
-        xyz="0 0 0" />
-    </joint> -->
-    <!-- <xacro:if value="${vision}">
-      <link name="${prefix}camera_link" />
-      <joint name="${prefix}camera_module" type="fixed">
-        <origin xyz="0 0.05639 -0.00305" rpy="3.14159265358979 3.14159265358979 0" />
-        <parent link="${prefix}end_effector_link" />
-        <child  link="${prefix}camera_link" />
-      </joint>
-      <link name="${prefix}camera_depth_frame" />
-      <joint name="${prefix}depth_module" type="fixed">
-        <origin xyz="0.0275 0.066 -0.00305" rpy="3.14159265358979 3.14159265358979 0" />
-        <parent link="${prefix}end_effector_link" />
-        <child  link="${prefix}camera_depth_frame" />
-      </joint>
-      <link name="${prefix}camera_color_frame" />
-      <joint name="${prefix}color_module" type="fixed">
-        <origin xyz="0 0.05639 -0.00305" rpy="3.14159265358979 3.14159265358979 0" />
-        <parent link="${prefix}end_effector_link" />
-        <child  link="${prefix}camera_color_frame" />
-      </joint>
-    </xacro:if> -->
-    <!-- <gazebo reference="${prefix}ft_sensor">
-        <provideFeedback>true</provideFeedback>
-        <disableFixedJointLumping>true</disableFixedJointLumping>
-        <preserveFixedJoint>true</preserveFixedJoint>
-    </gazebo>
-    <gazebo>
-        <plugin name="ft_sensor" filename="libgazebo_ros_ft_sensor.so">
-            <updateRate>100.0</updateRate>
-            <topicName>ft_sensor</topicName>
-            <jointName>${prefix}ft_sensor</jointName>
-        </plugin>
-    </gazebo> -->
   </xacro:macro>
 </robot>

File: kortex_description/robots/kortex_table.xacro (robot description, xacro)
@@ -22,32 +22,51 @@
             <link name="table">
                 <visual>
-                <geometry>
-                    <mesh filename="package://kortex_description/meshes/table/visual/table.dae"/>
-                </geometry>
+                    <origin xyz="0 0 0.01" rpy="1.5708 0 0" />
+                    <geometry>
+                        <mesh filename="package://kortex_description/meshes/environment/Table_v2.STL"/>
+                    </geometry>
                 </visual>
                 <collision>
-                <geometry>
-                    <mesh filename="package://kortex_description/meshes/table/collision/table.obj"/>
-                </geometry>
+                    <origin xyz="0 0 0" rpy="1.5708 0 0" />
+                    <geometry>
+                        <mesh filename="package://kortex_description/meshes/environment/Table_v2.STL"/>
+                    </geometry>
                 </collision>
             </link>
-              <link name="pelvis_link">
+            <link name="wall">
                 <visual>
-                <geometry>
-                    <mesh filename="package://kortex_description/meshes/pelvis/pelvis_new.dae" scale="0.001 0.001 0.001"/>
-                </geometry>
+                    <geometry>
+                        <mesh filename="package://kortex_description/meshes/environment/Wall.STL"/>
+                    </geometry>
                 </visual>
-                <!-- <collision>
-                <geometry>
-                    <mesh filename="package://kortex_description/meshes/pelvis/pelvis_new.dae" scale="0.001 0.001 0.001"/>
-                </geometry>
-                </collision> -->
+                <collision>
+                    <geometry>
+                        <mesh filename="package://kortex_description/meshes/environment/Wall.STL"/>
+                    </geometry>
+                </collision>
             </link>
+            <!-- <link name="pelvis_link">
+              <visual>
+              <geometry>
+                  <mesh filename="package://kortex_description/meshes/pelvis/pelvis_new.dae" scale="0.001 0.001 0.001"/>
+              </geometry>
+              </visual>
+              <collision>
+              <geometry>
+                  <mesh filename="package://kortex_description/meshes/pelvis/pelvis_new.dae" scale="0.001 0.001 0.001"/>
+              </geometry>
+              </collision>
+            </link> -->
             <joint name="world_joint" type="fixed">
                 <parent link="world"/>
                 <child link="table"/>
-                <origin rpy="0.0 0.0 0" xyz="0.0 0.0 -0.005"/>
+                <origin rpy="0.0 0.0 0.0" xyz="0.0 0.0 0.0"/>
             </joint>
-            <joint name="pelvis_joint" type="fixed">
+            <joint name="world2wall_joint" type="fixed">
+                <parent link="world"/>
+                <child link="wall"/>
+                <origin rpy="1.5708 0.0 1.5708" xyz="0.0 0.32 0.0"/>
+            </joint>
+            <!-- <joint name="pelvis_joint" type="fixed">
                 <parent link="table" />
                 <child link = "pelvis_link" />
@@ -55,14 +74,20 @@
                 <limit lower="-3.1416" upper="3.1416" effort="10" velocity="3"/>
                 <axis xyz="0 1 0"/>
-            </joint>
+            </joint> -->
             <joint name="table_joint" type="fixed">
+                <parent link="table" />
                 <child link="${prefix}base_link" />
-                <parent link="table" />
                 <origin xyz="0 0 0" rpy="0 0 0" />
             </joint>
-            <gazebo reference="pelvis">
+            <!-- <gazebo reference="pelvis">
+                <selfCollide>true</selfCollide>
+            </gazebo> -->
+            <gazebo reference="table">
                 <selfCollide>true</selfCollide>
             </gazebo>
-            <gazebo reference="table">
+            <gazebo reference="wall">
+                <selfCollide>true</selfCollide>
+            </gazebo>
+            <gazebo reference="${prefix}base_link">
                 <selfCollide>true</selfCollide>
             </gazebo>
@@ -81,39 +106,58 @@
         <!-- TODO: If the following is changed, need to change also in kortex_robot and in robot_model (Kortex Control) -->
         <xacro:if value="${not gripper}">
-            <link name="${prefix}ee_marker_frame"/>
-            <joint name="${prefix}ee_marker_frame_joint" type="fixed">
-                <origin xyz="0 0 0" rpy="-1.5708 0 0" />
+            <link name="${prefix}tool_frame">
+                <visual>
+                    <origin xyz="0 0 0" rpy="0 0 0" />
+                    <geometry>
+                    <mesh filename="package://kortex_description/arms/gen3/${dof}dof/meshes/ReamerHead.STL"/>
+                    </geometry>
+                    <material name="">
+                    <color rgba="0.75294 0.75294 0.75294 1" />
+                    </material>
+                </visual>
+                <collision>
+                    <origin xyz="0 0 0" rpy="0 0 0" />
+                    <geometry>
+                    <mesh filename="package://kortex_description/arms/gen3/${dof}dof/meshes/ReamerHead.STL"/>
+                    </geometry>
+                </collision>
+            </link>
+            <joint name="${prefix}tool_frame_joint" type="prismatic">
+                <origin xyz="0 0 -0.0915" rpy="0 0 0" />
                 <parent link="${prefix}${last_arm_link}" />
-                <child link="${prefix}ee_marker_frame" />
-                <axis xyz="0 0 0" />
+                <child link="${prefix}tool_frame" />
+                <axis xyz="0 0 1" />
+                <limit lower="-0.07" upper="0" effort="200" velocity="40" />
             </joint>
-            <link name="${prefix}tool_frame"/>
-            <joint name="${prefix}tool_frame_joint" type="fixed">
-                <origin xyz="-0.008480 -0.191619 0 " rpy="-1.5708 0 -0.7854" />
-                <parent link="${prefix}ee_marker_frame" />
-                <child link="${prefix}tool_frame" />
+            <link name="${prefix}reamer_head">
+                <visual>
+                    <origin xyz="0 0 0" rpy="0 0 0" />
+                    <geometry>
+                    <mesh filename="package://kortex_description/arms/gen3/${dof}dof/meshes/ReamingHead_56MM.STL"/>
+                    </geometry>
+                    <material name="">
+                    <color rgba="0.75294 0.75294 0.75294 1" />
+                    </material>
+                </visual>
+                <collision>
+                    <origin xyz="0 0 0" rpy="0 0 0" />
+                    <geometry>
+                    <mesh filename="package://kortex_description/arms/gen3/${dof}dof/meshes/ReamingHead_56MM.STL"/>
+                    </geometry>
+                </collision>
+            </link>
+            <joint name="${prefix}reamer_head_joint" type="fixed">
+                <origin xyz="0 0 0" rpy="0 0 0" />
+                <parent link="${prefix}tool_frame" />
+                <child link="${prefix}reamer_head" />
                 <axis xyz="0 0 0" />
             </joint>
             <link name="${prefix}tool_tip_frame"/>
             <joint name="${prefix}tool_tip_frame_joint" type="fixed">
-                <origin xyz="0 0 -0.023" rpy="0 0 0" />
-                <parent link="${prefix}tool_frame" />
+                <origin xyz="0 0 -0.028" rpy="0 0 0" />
+                <parent link="${prefix}reamer_head" />
                 <child link="${prefix}tool_tip_frame"/>
                 <axis xyz="0 0 0" />
             </joint>
-            <!-- <link name="${prefix}tool_tip_frame"/>
-            <joint name="${prefix}tool_tip_frame_joint" type="fixed">
-                <origin xyz="0 -0.16290848 0" rpy="-1.5708 0 0" />
-                <parent link="${prefix}ee_marker_frame" />
-                <child link="${prefix}tool_tip_frame" />
-                <axis xyz="0 0 0" />
-            </joint>
-            <link name="${prefix}tool_frame"/>
-            <joint name="${prefix}tool_frame_joint" type="fixed">
-                <origin xyz="0 0 0.023" rpy="0 0 0" />
-                <parent link="${prefix}tool_tip_frame" />
-                <child link="${prefix}tool_frame"/>
-                <axis xyz="0 0 0" />
-            </joint> -->
         </xacro:if>
         <!-- Load the Gazebo transmissions and gazebo_ros_control plugin -->
