Commit message: Updated urdf and modified arm controls to use tool frame tip (untested)

File: kortex_description/robots/kortex_table_old.xacro (robot description, xacro)
@@ -22,51 +22,32 @@
             <link name="table">
                 <visual>
-                    <origin xyz="0 0 0.01" rpy="1.5708 0 0" />
-                    <geometry>
-                        <mesh filename="package://kortex_description/meshes/environment/Table_v2.STL"/>
-                    </geometry>
+                <geometry>
+                    <mesh filename="package://kortex_description/meshes/table/visual/table.dae"/>
+                </geometry>
                 </visual>
                 <collision>
-                    <origin xyz="0 0 0" rpy="1.5708 0 0" />
-                    <geometry>
-                        <mesh filename="package://kortex_description/meshes/environment/Table_v2.STL"/>
-                    </geometry>
+                <geometry>
+                    <mesh filename="package://kortex_description/meshes/table/collision/table.obj"/>
+                </geometry>
                 </collision>
             </link>
-            <link name="wall">
+              <link name="pelvis_link">
                 <visual>
-                    <geometry>
-                        <mesh filename="package://kortex_description/meshes/environment/Wall.STL"/>
-                    </geometry>
+                <geometry>
+                    <mesh filename="package://kortex_description/meshes/pelvis/pelvis_new.dae" scale="0.001 0.001 0.001"/>
+                </geometry>
                 </visual>
-                <collision>
-                    <geometry>
-                        <mesh filename="package://kortex_description/meshes/environment/Wall.STL"/>
-                    </geometry>
-                </collision>
+                <!-- <collision>
+                <geometry>
+                    <mesh filename="package://kortex_description/meshes/pelvis/pelvis_new.dae" scale="0.001 0.001 0.001"/>
+                </geometry>
+                </collision> -->
             </link>
-            <!-- <link name="pelvis_link">
-              <visual>
-              <geometry>
-                  <mesh filename="package://kortex_description/meshes/pelvis/pelvis_new.dae" scale="0.001 0.001 0.001"/>
-              </geometry>
-              </visual>
-              <collision>
-              <geometry>
-                  <mesh filename="package://kortex_description/meshes/pelvis/pelvis_new.dae" scale="0.001 0.001 0.001"/>
-              </geometry>
-              </collision>
-            </link> -->
             <joint name="world_joint" type="fixed">
                 <parent link="world"/>
                 <child link="table"/>
-                <origin rpy="0.0 0.0 0.0" xyz="0.0 0.0 0.0"/>
+                <origin rpy="0.0 0.0 0" xyz="0.0 0.0 -0.005"/>
             </joint>
-            <joint name="world2wall_joint" type="fixed">
-                <parent link="world"/>
-                <child link="wall"/>
-                <origin rpy="1.5708 0.0 1.5708" xyz="0.0 0.32 0.0"/>
-            </joint>
-            <!-- <joint name="pelvis_joint" type="fixed">
+            <joint name="pelvis_joint" type="fixed">
                 <parent link="table" />
                 <child link = "pelvis_link" />
@@ -74,20 +55,14 @@
                 <limit lower="-3.1416" upper="3.1416" effort="10" velocity="3"/>
                 <axis xyz="0 1 0"/>
-            </joint> -->
+            </joint>
             <joint name="table_joint" type="fixed">
+                <child link="${prefix}base_link" />
                 <parent link="table" />
-                <child link="${prefix}base_link" />
                 <origin xyz="0 0 0" rpy="0 0 0" />
             </joint>
-            <!-- <gazebo reference="pelvis">
-                <selfCollide>true</selfCollide>
-            </gazebo> -->
-            <gazebo reference="table">
+            <gazebo reference="pelvis">
                 <selfCollide>true</selfCollide>
             </gazebo>
-            <gazebo reference="wall">
-                <selfCollide>true</selfCollide>
-            </gazebo>
-            <gazebo reference="${prefix}base_link">
+            <gazebo reference="table">
                 <selfCollide>true</selfCollide>
             </gazebo>
@@ -106,39 +81,58 @@
         <!-- TODO: If the following is changed, need to change also in kortex_robot and in robot_model (Kortex Control) -->
         <xacro:if value="${not gripper}">
-            <link name="${prefix}ee_marker_frame"/>
-            <joint name="${prefix}ee_marker_frame_joint" type="fixed">
-                <origin xyz="0 0 0" rpy="-1.5708 0 0" />
+            <link name="${prefix}tool_frame">
+                <visual>
+                    <origin xyz="0 0 0" rpy="0 0 0" />
+                    <geometry>
+                    <mesh filename="package://kortex_description/arms/gen3/${dof}dof/meshes/ReamerHead.STL"/>
+                    </geometry>
+                    <material name="">
+                    <color rgba="0.75294 0.75294 0.75294 1" />
+                    </material>
+                </visual>
+                <collision>
+                    <origin xyz="0 0 0" rpy="0 0 0" />
+                    <geometry>
+                    <mesh filename="package://kortex_description/arms/gen3/${dof}dof/meshes/ReamerHead.STL"/>
+                    </geometry>
+                </collision>
+            </link>
+            <joint name="${prefix}tool_frame_joint" type="prismatic">
+                <origin xyz="0 0 -0.0915" rpy="0 0 0" />
                 <parent link="${prefix}${last_arm_link}" />
-                <child link="${prefix}ee_marker_frame" />
-                <axis xyz="0 0 0" />
+                <child link="${prefix}tool_frame" />
+                <axis xyz="0 0 1" />
+                <limit lower="-0.07" upper="0" effort="200" velocity="40" />
             </joint>
-            <link name="${prefix}tool_frame"/>
-            <joint name="${prefix}tool_frame_joint" type="fixed">
-                <origin xyz="-0.008480 -0.191619 0 " rpy="-1.5708 0 -0.7854" />
-                <parent link="${prefix}ee_marker_frame" />
-                <child link="${prefix}tool_frame" />
+            <link name="${prefix}reamer_head">
+                <visual>
+                    <origin xyz="0 0 0" rpy="0 0 0" />
+                    <geometry>
+                    <mesh filename="package://kortex_description/arms/gen3/${dof}dof/meshes/ReamingHead_56MM.STL"/>
+                    </geometry>
+                    <material name="">
+                    <color rgba="0.75294 0.75294 0.75294 1" />
+                    </material>
+                </visual>
+                <collision>
+                    <origin xyz="0 0 0" rpy="0 0 0" />
+                    <geometry>
+                    <mesh filename="package://kortex_description/arms/gen3/${dof}dof/meshes/ReamingHead_56MM.STL"/>
+                    </geometry>
+                </collision>
+            </link>
+            <joint name="${prefix}reamer_head_joint" type="fixed">
+                <origin xyz="0 0 0" rpy="0 0 0" />
+                <parent link="${prefix}tool_frame" />
+                <child link="${prefix}reamer_head" />
                 <axis xyz="0 0 0" />
             </joint>
             <link name="${prefix}tool_tip_frame"/>
             <joint name="${prefix}tool_tip_frame_joint" type="fixed">
-                <origin xyz="0 0 -0.023" rpy="0 0 0" />
-                <parent link="${prefix}tool_frame" />
+                <origin xyz="0 0 -0.028" rpy="0 0 0" />
+                <parent link="${prefix}reamer_head" />
                 <child link="${prefix}tool_tip_frame"/>
                 <axis xyz="0 0 0" />
             </joint>
-            <!-- <link name="${prefix}tool_tip_frame"/>
-            <joint name="${prefix}tool_tip_frame_joint" type="fixed">
-                <origin xyz="0 -0.16290848 0" rpy="-1.5708 0 0" />
-                <parent link="${prefix}ee_marker_frame" />
-                <child link="${prefix}tool_tip_frame" />
-                <axis xyz="0 0 0" />
-            </joint>
-            <link name="${prefix}tool_frame"/>
-            <joint name="${prefix}tool_frame_joint" type="fixed">
-                <origin xyz="0 0 0.023" rpy="0 0 0" />
-                <parent link="${prefix}tool_tip_frame" />
-                <child link="${prefix}tool_frame"/>
-                <axis xyz="0 0 0" />
-            </joint> -->
         </xacro:if>
         <!-- Load the Gazebo transmissions and gazebo_ros_control plugin -->

Commit message: Fixing arm calibration

File: kortex_control/arm_description/robot_model.xacro (robot description, xacro)
@@ -47,5 +47,5 @@
             <origin xyz="0 0 0" rpy="0 0 0" />
             <geometry>
-            <mesh filename="package://kortex_description/arms/gen3/$(arg dof)dof/meshes/ReamingHead_56MM.STL"/>
+            <mesh filename="package://kortex_description/arms/gen3/$(arg dof)dof/meshes/ReamingHead_48MM.STL"/>
             </geometry>
             <material name="">
@@ -56,5 +56,5 @@
             <origin xyz="0 0 0" rpy="0 0 0" />
             <geometry>
-            <mesh filename="package://kortex_description/arms/gen3/$(arg dof)dof/meshes/ReamingHead_56MM.STL"/>
+            <mesh filename="package://kortex_description/arms/gen3/$(arg dof)dof/meshes/ReamingHead_48MM.STL"/>
             </geometry>
         </collision>
@@ -68,5 +68,5 @@
     <link name="$(arg prefix)tool_tip_frame"/>
     <joint name="$(arg prefix)tool_tip_frame_joint" type="fixed">
-        <origin xyz="0 0 -0.028" rpy="0 0 0" />
+        <origin xyz="0 0 -0.024" rpy="0 0 0" />
         <parent link="$(arg prefix)reamer_head" />
         <child link="$(arg prefix)tool_tip_frame"/>

File: kortex_description/arms/gen3/7dof/urdf/gen3_macro.xacro (robot description, xacro)
@@ -331,4 +331,5 @@
     <link name="${prefix}ee_marker_frame"/>
     <joint name="${prefix}ee_marker_frame_joint" type="fixed">
+        <!-- <origin xyz="0.034 0.0457193 0.14223149" rpy="0 -1.570796327 0" /> -->
         <origin xyz="0.042 0.0417193 0.14523149" rpy="0 -1.570796327 0" />
         <!-- <origin xyz="0 0.01025305 0.17316221" rpy="0 -1.570796327 0" /> -->
@@ -339,4 +340,5 @@
     <link name="${prefix}ee_reamer_hole"/>
     <joint name="${prefix}ee_reamer_hole_joint" type="fixed">
+        <!-- <origin xyz="0.03093072 -0.02746625 0.034" rpy="-1.570796327 -1.570796327 0.7853981635" /> -->
         <origin xyz="0.02793072 -0.03146625 0.042" rpy="-1.570796327 -1.570796327 0.7853981635" />
         <parent link="${prefix}ee_marker_frame" />

File: kortex_description/robots/gen3.xacro (robot description, xacro)
@@ -8,5 +8,6 @@
     <xacro:arg name="sim" default="false" />
     <xacro:arg name="prefix" default="" />
+    <xacro:arg name="ee_joint_fixed" default="true" />
     <xacro:include filename="$(find kortex_description)/robots/kortex_table.xacro" />
-    <xacro:load_robot arm="$(arg arm)" gripper="$(arg gripper)" dof="$(arg dof)" vision="$(arg vision)" sim="$(arg sim)" prefix="$(arg prefix)" />
+    <xacro:load_robot arm="$(arg arm)" gripper="$(arg gripper)" dof="$(arg dof)" vision="$(arg vision)" sim="$(arg sim)" prefix="$(arg prefix)" ee_joint_fixed="$(arg ee_joint_fixed)" />
 </robot>

File: kortex_description/robots/kortex_table.xacro (robot description, xacro)
@@ -2,5 +2,5 @@
 <!-- use this to generate urdf -->
 <robot xmlns:xacro="http://ros.org/wiki/xacro">
-    <xacro:macro name="load_robot" params="arm gripper dof vision sim prefix">
+    <xacro:macro name="load_robot" params="arm gripper dof vision sim prefix ee_joint_fixed">
         <!-- Files to include -->
         <xacro:include filename="$(find kortex_description)/arms/${arm}/${dof}dof/urdf/${arm}_macro.xacro" />
@@ -123,16 +123,27 @@
                 </collision>
             </link>
-            <joint name="${prefix}tool_frame_joint" type="prismatic">
-                <origin xyz="0 0 -0.0915" rpy="0 0 0" />
-                <parent link="${prefix}${last_arm_link}" />
-                <child link="${prefix}tool_frame" />
-                <axis xyz="0 0 1" />
-                <limit lower="-0.07" upper="0" effort="200" velocity="40" />
-            </joint>
+            <xacro:if value="${ee_joint_fixed}">
+                <joint name="${prefix}tool_frame_joint" type="fixed">
+                    <origin xyz="0 0 -0.0915" rpy="0 0 0" />
+                    <parent link="${prefix}${last_arm_link}" />
+                    <child link="${prefix}tool_frame" />
+                    <axis xyz="0 0 1" />
+                    <limit lower="-0.07" upper="0" effort="200" velocity="40" />
+                </joint>
+            </xacro:if>
+            <xacro:unless value="${ee_joint_fixed}">
+                <joint name="${prefix}tool_frame_joint" type="prismatic">
+                    <origin xyz="0 0 -0.0915" rpy="0 0 0" />
+                    <parent link="${prefix}${last_arm_link}" />
+                    <child link="${prefix}tool_frame" />
+                    <axis xyz="0 0 1" />
+                    <limit lower="-0.07" upper="0" effort="200" velocity="40" />
+                </joint>
+            </xacro:unless>
             <link name="${prefix}reamer_head">
                 <visual>
                     <origin xyz="0 0 0" rpy="0 0 0" />
                     <geometry>
-                    <mesh filename="package://kortex_description/arms/gen3/${dof}dof/meshes/ReamingHead_56MM.STL"/>
+                    <mesh filename="package://kortex_description/arms/gen3/${dof}dof/meshes/ReamingHead_48MM.STL"/>
                     </geometry>
                     <material name="">
@@ -143,5 +154,5 @@
                     <origin xyz="0 0 0" rpy="0 0 0" />
                     <geometry>
-                    <mesh filename="package://kortex_description/arms/gen3/${dof}dof/meshes/ReamingHead_56MM.STL"/>
+                    <mesh filename="package://kortex_description/arms/gen3/${dof}dof/meshes/ReamingHead_48MM.STL"/>
                     </geometry>
                 </collision>
@@ -155,5 +166,5 @@
             <link name="${prefix}tool_tip_frame"/>
             <joint name="${prefix}tool_tip_frame_joint" type="fixed">
-                <origin xyz="0 0 -0.028" rpy="0 0 0" />
+                <origin xyz="0 0 -0.024" rpy="0 0 0" />
                 <parent link="${prefix}reamer_head" />
                 <child link="${prefix}tool_tip_frame"/>

Commit message: Fixed online calibration and urdf

File: kortex_control/arm_description/robot_model.xacro (robot description, xacro)
@@ -37,5 +37,5 @@
     </link>
     <joint name="$(arg prefix)tool_frame_joint" type="fixed">
-        <origin xyz="0 0 -0.0915" rpy="0 0 0" />
+        <origin xyz="0 0 -0.0858" rpy="0 0 0" />
         <parent link="$(arg prefix)${last_arm_link}" />
         <child link="$(arg prefix)tool_frame" />

File: kortex_control/arm_description/test.urdf (robot description, URDF)
Before this commit: robot gen3, 16 links, 15 joints
Joints:
- joint tool_frame_joint: origin xyz=0 0 -0.0915 rpy=0 0 0 -> xyz=0 0 -0.0858 rpy=0 0 0

File: kortex_description/robots/kortex_table.xacro (robot description, xacro)
@@ -125,5 +125,5 @@
             <xacro:if value="${ee_joint_fixed}">
                 <joint name="${prefix}tool_frame_joint" type="fixed">
-                    <origin xyz="0 0 -0.0915" rpy="0 0 0" />
+                    <origin xyz="0 0 -0.0858" rpy="0 0 0" />
                     <parent link="${prefix}${last_arm_link}" />
                     <child link="${prefix}tool_frame" />
@@ -134,5 +134,5 @@
             <xacro:unless value="${ee_joint_fixed}">
                 <joint name="${prefix}tool_frame_joint" type="prismatic">
-                    <origin xyz="0 0 -0.0915" rpy="0 0 0" />
+                    <origin xyz="0 0 -0.0858" rpy="0 0 0" />
                     <parent link="${prefix}${last_arm_link}" />
                     <child link="${prefix}tool_frame" />

File: kortex_description/robots/kortex_table_collision.xacro (robot description, xacro)
@@ -125,5 +125,5 @@
             <xacro:if value="${ee_joint_fixed}">
                 <joint name="${prefix}tool_frame_joint" type="fixed">
-                    <origin xyz="0 0 -0.0915" rpy="0 0 0" />
+                    <origin xyz="0 0 -0.0858" rpy="0 0 0" />
                     <parent link="${prefix}${last_arm_link}" />
                     <child link="${prefix}tool_frame" />
@@ -134,5 +134,5 @@
             <xacro:unless value="${ee_joint_fixed}">
                 <joint name="${prefix}tool_frame_joint" type="prismatic">
-                    <origin xyz="0 0 -0.0915" rpy="0 0 0" />
+                    <origin xyz="0 0 -0.0858" rpy="0 0 0" />
                     <parent link="${prefix}${last_arm_link}" />
                     <child link="${prefix}tool_frame" />

File: kortex_description/robots/kortex_table_old.xacro (robot description, xacro)
@@ -99,5 +99,5 @@
             </link>
             <joint name="${prefix}tool_frame_joint" type="prismatic">
-                <origin xyz="0 0 -0.0915" rpy="0 0 0" />
+                <origin xyz="0 0 -0.0858" rpy="0 0 0" />
                 <parent link="${prefix}${last_arm_link}" />
                 <child link="${prefix}tool_frame" />

Commit message: urdf updated with new ee length

File: kortex_control/arm_description/robot_model.xacro (robot description, xacro)
@@ -37,5 +37,5 @@
     </link>
     <joint name="$(arg prefix)tool_frame_joint" type="fixed">
-        <origin xyz="0 0 -0.0858" rpy="0 0 0" />
+        <origin xyz="0 0 -0.087" rpy="0 0 0" />
         <parent link="$(arg prefix)${last_arm_link}" />
         <child link="$(arg prefix)tool_frame" />

File: kortex_control/arm_description/test.urdf (robot description, URDF)
Before this commit: robot gen3, 16 links, 15 joints
Joints:
- joint tool_frame_joint: origin xyz=0 0 -0.0858 rpy=0 0 0 -> xyz=0 0 -0.087 rpy=0 0 0

File: kortex_description/robots/kortex_table.xacro (robot description, xacro)
@@ -125,5 +125,5 @@
             <xacro:if value="${ee_joint_fixed}">
                 <joint name="${prefix}tool_frame_joint" type="fixed">
-                    <origin xyz="0 0 -0.0858" rpy="0 0 0" />
+                    <origin xyz="0 0 -0.087" rpy="0 0 0" />
                     <parent link="${prefix}${last_arm_link}" />
                     <child link="${prefix}tool_frame" />
@@ -134,5 +134,5 @@
             <xacro:unless value="${ee_joint_fixed}">
                 <joint name="${prefix}tool_frame_joint" type="prismatic">
-                    <origin xyz="0 0 -0.0858" rpy="0 0 0" />
+                    <origin xyz="0 0 -0.087" rpy="0 0 0" />
                     <parent link="${prefix}${last_arm_link}" />
                     <child link="${prefix}tool_frame" />

File: kortex_description/robots/kortex_table_collision.xacro (robot description, xacro)
@@ -125,5 +125,5 @@
             <xacro:if value="${ee_joint_fixed}">
                 <joint name="${prefix}tool_frame_joint" type="fixed">
-                    <origin xyz="0 0 -0.0858" rpy="0 0 0" />
+                    <origin xyz="0 0 -0.087" rpy="0 0 0" />
                     <parent link="${prefix}${last_arm_link}" />
                     <child link="${prefix}tool_frame" />
@@ -134,5 +134,5 @@
             <xacro:unless value="${ee_joint_fixed}">
                 <joint name="${prefix}tool_frame_joint" type="prismatic">
-                    <origin xyz="0 0 -0.0858" rpy="0 0 0" />
+                    <origin xyz="0 0 -0.087" rpy="0 0 0" />
                     <parent link="${prefix}${last_arm_link}" />
                     <child link="${prefix}tool_frame" />

File: kortex_description/robots/kortex_table_old.xacro (robot description, xacro)
@@ -99,5 +99,5 @@
             </link>
             <joint name="${prefix}tool_frame_joint" type="prismatic">
-                <origin xyz="0 0 -0.0858" rpy="0 0 0" />
+                <origin xyz="0 0 -0.087" rpy="0 0 0" />
                 <parent link="${prefix}${last_arm_link}" />
                 <child link="${prefix}tool_frame" />
