Commit message: FVD day tuning

File: kortex_control/arm_description/robot_model.xacro (robot description, xacro)
@@ -47,5 +47,5 @@
             <origin xyz="0 0 0" rpy="0 0 0" />
             <geometry>
-            <mesh filename="package://kortex_description/arms/gen3/$(arg dof)dof/meshes/ReamingHead_48MM.stl"/>
+            <mesh filename="package://kortex_description/arms/gen3/$(arg dof)dof/meshes/ReamingHead_56MM.stl"/>
             </geometry>
             <material name="">
@@ -56,5 +56,5 @@
             <origin xyz="0 0 0" rpy="0 0 0" />
             <geometry>
-            <mesh filename="package://kortex_description/arms/gen3/$(arg dof)dof/meshes/ReamingHead_48MM.stl"/>
+            <mesh filename="package://kortex_description/arms/gen3/$(arg dof)dof/meshes/ReamingHead_56MM.stl"/>
             </geometry>
         </collision>
@@ -68,5 +68,5 @@
     <link name="$(arg prefix)tool_tip_frame"/>
     <joint name="$(arg prefix)tool_tip_frame_joint" type="fixed">
-        <origin xyz="0 0 -0.024" rpy="0 0 0" />
+        <origin xyz="0 0 -0.028" rpy="0 0 0" />
         <parent link="$(arg prefix)reamer_head" />
         <child link="$(arg prefix)tool_tip_frame"/>

File: kortex_control/arm_description/test.urdf (robot description, URDF)
Before this commit: robot gen3, 16 links, 15 joints
Joints:
- joint tool_tip_frame_joint: origin xyz=0 0 -0.024 rpy=0 0 0 -> xyz=0 0 -0.028 rpy=0 0 0

File: kortex_description/robots/kortex_table.xacro (robot description, xacro)
@@ -145,5 +145,5 @@
                     <origin xyz="0 0 0" rpy="0 0 0" />
                     <geometry>
-                    <mesh filename="package://kortex_description/arms/gen3/${dof}dof/meshes/ReamingHead_48MM.stl"/>
+                    <mesh filename="package://kortex_description/arms/gen3/${dof}dof/meshes/ReamingHead_56MM.stl"/>
                     </geometry>
                     <material name="">
@@ -154,5 +154,5 @@
                     <origin xyz="0 0 0" rpy="0 0 0" />
                     <geometry>
-                    <mesh filename="package://kortex_description/arms/gen3/${dof}dof/meshes/ReamingHead_48MM.stl"/>
+                    <mesh filename="package://kortex_description/arms/gen3/${dof}dof/meshes/ReamingHead_56MM.stl"/>
                     </geometry>
                 </collision>
@@ -166,5 +166,5 @@
             <link name="${prefix}tool_tip_frame"/>
             <joint name="${prefix}tool_tip_frame_joint" type="fixed">
-                <origin xyz="0 0 -0.024" rpy="0 0 0" />
+                <origin xyz="0 0 -0.028" rpy="0 0 0" />
                 <parent link="${prefix}reamer_head" />
                 <child link="${prefix}tool_tip_frame"/>

File: kortex_description/robots/kortex_table_collision.xacro (robot description, xacro)
@@ -145,5 +145,5 @@
                     <origin xyz="0 0 0" rpy="0 0 0" />
                     <geometry>
-                    <mesh filename="package://kortex_description/arms/gen3/${dof}dof/meshes/ReamingHead_48MM.stl"/>
+                    <mesh filename="package://kortex_description/arms/gen3/${dof}dof/meshes/ReamingHead_56MM.stl"/>
                     </geometry>
                     <material name="">
@@ -154,5 +154,5 @@
                     <origin xyz="0 0 0" rpy="0 0 0" />
                     <geometry>
-                    <mesh filename="package://kortex_description/arms/gen3/${dof}dof/meshes/ReamingHead_48MM.stl"/>
+                    <mesh filename="package://kortex_description/arms/gen3/${dof}dof/meshes/ReamingHead_56MM.stl"/>
                     </geometry>
                 </collision>
@@ -166,5 +166,5 @@
             <link name="${prefix}tool_tip_frame"/>
             <joint name="${prefix}tool_tip_frame_joint" type="fixed">
-                <origin xyz="0 0 -0.024" rpy="0 0 0" />
+                <origin xyz="0 0 -0.028" rpy="0 0 0" />
                 <parent link="${prefix}reamer_head" />
                 <child link="${prefix}tool_tip_frame"/>

File: kortex_description/robots/kortex_table_old.xacro (robot description, xacro)
@@ -109,5 +109,5 @@
                     <origin xyz="0 0 0" rpy="0 0 0" />
                     <geometry>
-                    <mesh filename="package://kortex_description/arms/gen3/${dof}dof/meshes/ReamingHead_48MM.stl"/>
+                    <mesh filename="package://kortex_description/arms/gen3/${dof}dof/meshes/ReamingHead_56MM.stl"/>
                     </geometry>
                     <material name="">
@@ -118,5 +118,5 @@
                     <origin xyz="0 0 0" rpy="0 0 0" />
                     <geometry>
-                    <mesh filename="package://kortex_description/arms/gen3/${dof}dof/meshes/ReamingHead_48MM.stl"/>
+                    <mesh filename="package://kortex_description/arms/gen3/${dof}dof/meshes/ReamingHead_56MM.stl"/>
                     </geometry>
                 </collision>
@@ -130,5 +130,5 @@
             <link name="${prefix}tool_tip_frame"/>
             <joint name="${prefix}tool_tip_frame_joint" type="fixed">
-                <origin xyz="0 0 -0.024" rpy="0 0 0" />
+                <origin xyz="0 0 -0.028" rpy="0 0 0" />
                 <parent link="${prefix}reamer_head" />
                 <child link="${prefix}tool_tip_frame"/>

Commit message: Changed from 56MM to 48MM reamer head

File: kortex_control/arm_description/robot_model.xacro (robot description, xacro)
@@ -47,5 +47,5 @@
             <origin xyz="0 0 0" rpy="0 0 0" />
             <geometry>
-            <mesh filename="package://kortex_description/arms/gen3/$(arg dof)dof/meshes/ReamingHead_56MM.stl"/>
+            <mesh filename="package://kortex_description/arms/gen3/$(arg dof)dof/meshes/ReamingHead_48MM.stl"/>
             </geometry>
             <material name="">
@@ -56,5 +56,5 @@
             <origin xyz="0 0 0" rpy="0 0 0" />
             <geometry>
-            <mesh filename="package://kortex_description/arms/gen3/$(arg dof)dof/meshes/ReamingHead_56MM.stl"/>
+            <mesh filename="package://kortex_description/arms/gen3/$(arg dof)dof/meshes/ReamingHead_48MM.stl"/>
             </geometry>
         </collision>
@@ -68,5 +68,5 @@
     <link name="$(arg prefix)tool_tip_frame"/>
     <joint name="$(arg prefix)tool_tip_frame_joint" type="fixed">
-        <origin xyz="0 0 -0.028" rpy="0 0 0" />
+        <origin xyz="0 0 -0.024" rpy="0 0 0" />
         <parent link="$(arg prefix)reamer_head" />
         <child link="$(arg prefix)tool_tip_frame"/>

File: kortex_description/robots/kortex_table.xacro (robot description, xacro)
@@ -145,5 +145,5 @@
                     <origin xyz="0 0 0" rpy="0 0 0" />
                     <geometry>
-                    <mesh filename="package://kortex_description/arms/gen3/${dof}dof/meshes/ReamingHead_56MM.stl"/>
+                    <mesh filename="package://kortex_description/arms/gen3/${dof}dof/meshes/ReamingHead_48MM.stl"/>
                     </geometry>
                     <material name="">
@@ -154,5 +154,5 @@
                     <origin xyz="0 0 0" rpy="0 0 0" />
                     <geometry>
-                    <mesh filename="package://kortex_description/arms/gen3/${dof}dof/meshes/ReamingHead_56MM.stl"/>
+                    <mesh filename="package://kortex_description/arms/gen3/${dof}dof/meshes/ReamingHead_48MM.stl"/>
                     </geometry>
                 </collision>
@@ -166,5 +166,5 @@
             <link name="${prefix}tool_tip_frame"/>
             <joint name="${prefix}tool_tip_frame_joint" type="fixed">
-                <origin xyz="0 0 -0.028" rpy="0 0 0" />
+                <origin xyz="0 0 -0.024" rpy="0 0 0" />
                 <parent link="${prefix}reamer_head" />
                 <child link="${prefix}tool_tip_frame"/>

File: kortex_description/robots/kortex_table_collision.xacro (robot description, xacro)
@@ -145,5 +145,5 @@
                     <origin xyz="0 0 0" rpy="0 0 0" />
                     <geometry>
-                    <mesh filename="package://kortex_description/arms/gen3/${dof}dof/meshes/ReamingHead_56MM.stl"/>
+                    <mesh filename="package://kortex_description/arms/gen3/${dof}dof/meshes/ReamingHead_48MM.stl"/>
                     </geometry>
                     <material name="">
@@ -154,5 +154,5 @@
                     <origin xyz="0 0 0" rpy="0 0 0" />
                     <geometry>
-                    <mesh filename="package://kortex_description/arms/gen3/${dof}dof/meshes/ReamingHead_56MM.stl"/>
+                    <mesh filename="package://kortex_description/arms/gen3/${dof}dof/meshes/ReamingHead_48MM.stl"/>
                     </geometry>
                 </collision>
@@ -166,5 +166,5 @@
             <link name="${prefix}tool_tip_frame"/>
             <joint name="${prefix}tool_tip_frame_joint" type="fixed">
-                <origin xyz="0 0 -0.028" rpy="0 0 0" />
+                <origin xyz="0 0 -0.024" rpy="0 0 0" />
                 <parent link="${prefix}reamer_head" />
                 <child link="${prefix}tool_tip_frame"/>
